File: pcb/FightKey.kicad_pcb (KiCad board)
At the start: 2 copper layers, 201.9 x 85.1 mm, 29 parts, among them J1 Conn_01x016_Male

Commit message: Converted to slimmer, openable model with split design (#1)
* Remade PCB to be split and include Pico in design

* Removed stray trace

* Restarted enclosure and modeled out new board left side as a reference

* Fixed missing connection (will have to hotwire physically :(

* Added bottom of enclosure (not done) and modeled right pcb board

* Added top-left of enclosure, left-side rounding, and screw holes

* Added top-right and fixed minor issues. Design complete

* Fixed the keybindings to match expected

* Turned off sys clock increase as it seems to break new pico for some reason

* Readded overclocking, but a decreased amount

* Reworked model polish (screw holes and roundedness stuff

* Fixed key bindings

* Fixed key bindings

* Updated model to fix print issue and increase screw size on incorrect hole

* Fixed some model issues and finished wide version
Parts:
- added J2: Conn_01x08_Male, Connector_PinHeader_2.54mm:PinHeader_1x08_P2.54mm_Vertical, F.Cu at (136.5, 90.2)
- added U1: Pico, MCU_RaspberryPi_and_Boards:RPi_Pico_SMD_TH, F.Cu at (158.8, 51.4)
- AK_BTN1: renamed from S456; footprint ECAD:MX1AE1NW -> SamacSys_Parts:MX1AE1NW
- AP_BT1: renamed from S123; footprint ECAD:MX1AE1NW -> SamacSys_Parts:MX1AE1NW
- DOWN_BTN1: renamed from SD1; footprint ECAD:MX1AE1NW -> SamacSys_Parts:MX1AE1NW
- HK_BTN1: renamed from S3; footprint ECAD:MX1AE1NW -> SamacSys_Parts:MX1AE1NW
- HP_BTN1: renamed from S6; footprint ECAD:MX1AE1NW -> SamacSys_Parts:MX1AE1NW
- J1: value Conn_01x016_Male -> Conn_01x08_Male; footprint Connector_PinHeader_2.54mm:PinHeader_1x16_P2.54mm_Vertical -> Connector_PinHeader_2.54mm:PinHeader_1x08_P2.54mm_Vertical
- LEFT_BTN1: renamed from SL1; footprint ECAD:MX1AE1NW -> SamacSys_Parts:MX1AE1NW
- LK_BTN1: renamed from S1; footprint ECAD:MX1AE1NW -> SamacSys_Parts:MX1AE1NW
- LP_BTN1: renamed from S4; footprint ECAD:MX1AE1NW -> SamacSys_Parts:MX1AE1NW
- MK_BTN1: renamed from S2; footprint ECAD:MX1AE1NW -> SamacSys_Parts:MX1AE1NW
- MP_BTN1: renamed from S5; footprint ECAD:MX1AE1NW -> SamacSys_Parts:MX1AE1NW
- RIGHT_BTN1: renamed from SR1; footprint ECAD:MX1AE1NW -> SamacSys_Parts:MX1AE1NW
- SELECT_BTN1: renamed from SS1; footprint ECAD:MX1AE1NW -> SamacSys_Parts:MX1AE1NW
- START_BTN1: renamed from SE1; footprint ECAD:MX1AE1NW -> SamacSys_Parts:MX1AE1NW
- UP_BTN1: renamed from SU1; footprint ECAD:MX1AE1NW -> SamacSys_Parts:MX1AE1NW
- moved R_P4 157.5 mm to (262.2, 41.3)
- moved R_K4 156.9 mm to (262.3, 79.4)
- moved R_P3 139.5 mm to (240.7, 31.8)
- moved R_K3 136.1 mm to (240.6, 70.5)
- moved R_P2 116.7 mm to (218.4, 31.8)
- moved J1 114.2 mm to (124.5, 90.2), turned to 0 degrees
- moved R_K2 113.5 mm to (218.4, 70.5)
- moved R_START1 99.6 mm to (123.2, 31.8)
- moved R_P1 94.0 mm to (196.8, 49.5)
- moved R_K1 91.5 mm to (196.8, 88.3)
- moved R_DOWN1 62.0 mm to (58.4, 99.7)
- moved R_RIGHT1 55.1 mm to (79.4, 75.6)
- moved AK_BTN1 52.1 mm to (255.9, 88.9)
- moved AP_BT1 52.1 mm to (255.9, 50.2)
- moved HK_BTN1 52.1 mm to (234.3, 80.0)
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- renumbered R2 to R_DOWN1, R7 to R_K1, R8 to R_K2, R9 to R_K3, R14 to R_K4, R3 to R_LEFT1, R11 to R_P1, R12 to R_P2, R13 to R_P3, R10 to R_P4, R4 to R_RIGHT1, R6 to R_SELECT1, R5 to R_START1, R1 to R_UP1
Connections:
- net /DOWN renamed /DOWNL
- net /ENTER renamed /STARTL
- net /LEFT renamed /LEFTL
- net /RIGHT renamed /RIGHTL
- net /SHIFT renamed /SELECTL
- net /UP renamed /UPL
- AK_BTN1 pad 2: /NENTER -> /AK
- AP_BT1 pad 2: /NPLUS -> /AP
- DOWN_BTN1 pad 1: /VCC -> /VCCL
- HK_BTN1 pad 2: /N3 -> /HK
- HP_BTN1 pad 2: /N6 -> /HP
- J1 pad 7: /N1 -> /VCCL
- J1 pad 8: /N2 -> /GNDL
- LEFT_BTN1 pad 1: /VCC -> /VCCL
- LK_BTN1 pad 2: /N1 -> /LK
- LP_BTN1 pad 2: /N4 -> /LP
- MK_BTN1 pad 2: /N2 -> /MK
- MP_BTN1 pad 2: /N5 -> /MP
- RIGHT_BTN1 pad 1: /VCC -> /VCCL
- R_DOWN1 pad 2: /GND -> /GNDL
- R_K1 pad 1: /N1 -> /LK
- R_K2 pad 1: /N2 -> /MK
- R_K3 pad 1: /N3 -> /HK
- R_K4 pad 1: /NENTER -> /AK
- R_LEFT1 pad 2: /GND -> /GNDL
- R_P1 pad 1: /N4 -> /LP
- R_P2 pad 1: /N5 -> /MP
- R_P3 pad 1: /N6 -> /HP
- R_P4 pad 1: /NPLUS -> /AP
- R_RIGHT1 pad 2: /GND -> /GNDL
- R_SELECT1 pad 2: /GND -> /GNDL
- R_START1 pad 2: /GND -> /GNDL
- R_UP1 pad 2: /GND -> /GNDL
- SELECT_BTN1 pad 1: /VCC -> /VCCL
- START_BTN1 pad 1: /VCC -> /VCCL
- UP_BTN1 pad 1: /VCC -> /VCCL
Routing:
- net /GNDL: track 0.00 -> 308.2 mm
- net /VCCL: track 0.00 -> 204.7 mm
- net /NENTER: track 191.4 -> 0.00 mm, vias 3 -> 0
- net /NPLUS: track 175.4 -> 0.00 mm, vias 1 -> 0
- net /N3: track 171.7 -> 0.00 mm, vias 2 -> 0
- net /AP: track 0.00 -> 158.4 mm, vias 0 -> 3
- net /N6: track 157.2 -> 0.00 mm, vias 3 -> 0
- net /N2: track 149.2 -> 0.00 mm, vias 3 -> 0
- net /GND: track 155.7 -> 291.4 mm, vias 0 -> 3
- net /HK: track 0.00 -> 133.9 mm, vias 0 -> 1
- net /N1: track 133.4 -> 0.00 mm, vias 2 -> 0
- net /N5: track 132.8 -> 0.00 mm, vias 2 -> 0
- net /HP: track 0.00 -> 124.6 mm, vias 0 -> 1
- net /N4: track 114.8 -> 0.00 mm, vias 2 -> 0
- net /VCC: track 409.7 -> 297.8 mm, vias 4 -> 1
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Other:
- board size 201.9 x 85.1 mm -> 254 x 85.1 mm
- board text added: "Create by Dylan Turner"
